Commit message: update 7.31

File: mani_skill/assets/robots/piper/piper_mplib.urdf (robot description, URDF)
Before this commit: robot piper, 11 links, 10 joints
Links:
- link base_link: geometry collision mesh filename=meshes/base_link.STL; visual mesh filename=meshes/base_link.STL
- link gripper_base: geometry collision mesh filename=meshes/gripper_base.STL; visual mesh filename=meshes/gripper_base.STL
- link link1: geometry collision mesh filename=meshes/link1.STL; visual mesh filename=meshes/link1.STL
- link link2: geometry collision mesh filename=meshes/link2.STL; visual mesh filename=meshes/link2.STL
- link link3: geometry collision mesh filename=meshes/link3.STL; visual mesh filename=meshes/link3.STL
- link link4: geometry collision mesh filename=meshes/link4.STL; visual mesh filename=meshes/link4.STL
- link link5: geometry collision mesh filename=meshes/link5.STL; visual mesh filename=meshes/link5.STL
- link link6: geometry collision mesh filename=meshes/link6.STL; visual mesh filename=meshes/link6.STL
- link link7: geometry collision mesh filename=meshes/link7.STL; visual mesh filename=meshes/link7.STL
- link link8: geometry collision mesh filename=meshes/link8.STL; visual mesh filename=meshes/link8.STL

File: mani_skill/assets/robots/piper/piper_old.urdf (robot description, URDF)
Before this commit: robot piper, 11 links, 10 joints
Links:
- link base_link: geometry collision mesh filename=meshes/base_link.STL; visual mesh filename=meshes/base_link.STL
- link gripper_base: geometry collision mesh filename=meshes/gripper_base.STL; visual mesh filename=meshes/gripper_base.STL
- link link1: geometry collision mesh filename=meshes/link1.STL; visual mesh filename=meshes/link1.STL
- link link2: geometry collision mesh filename=meshes/link2.STL; visual mesh filename=meshes/link2.STL
- link link3: geometry collision mesh filename=meshes/link3.STL; visual mesh filename=meshes/link3.STL
- link link4: geometry collision mesh filename=meshes/link4.STL; visual mesh filename=meshes/link4.STL
- link link5: geometry collision mesh filename=meshes/link5.STL; visual mesh filename=meshes/link5.STL
- link link6: geometry collision mesh filename=meshes/link6.STL; visual mesh filename=meshes/link6.STL
- link link7: geometry collision mesh filename=meshes/link7.STL; visual mesh filename=meshes/link7.STL
- link link8: geometry collision mesh filename=meshes/link8.STL; visual mesh filename=meshes/link8.STL
Joints:
- joint joint7: limit lower=0 upper=0.035 effort=100 velocity=1 -> lower=0 upper=0.035 effort=10 velocity=1
- joint joint8: limit lower=-0.035 upper=0 effort=100 velocity=1 -> lower=-0.035 upper=0 effort=10 velocity=1
