Commit message: 实现cobot抓取放置任务同步和异步执行

File: mani_skill/assets/robots/piper/piper_dual_arm_test.urdf (robot description, URDF)
Before this commit: robot piper, 11 links, 10 joints
Links:
- removed link dummy_link
- removed link gripper_base
- removed link link1
- removed link link2
- removed link link3
- removed link link4
- removed link link5
- removed link link6
- removed link link7
- removed link link8
- added link left_base_link, mass 0.097868; collision mesh filename=package://meshes/base_link.STL; visual mesh filename=package://meshes/base_link.STL
- added link left_camera_link, mass 0.001; visual box size=0.01 0.01 0.01
- added link left_link1, mass 0.097868; collision mesh filename=package://meshes/link1.STL; visual mesh filename=package://meshes/link1.STL
- added link left_link2, mass 0.290889; collision mesh filename=package://meshes/link2.STL; visual mesh filename=package://meshes/link2.STL
- added link left_link3, mass 0.290848; collision mesh filename=package://meshes/link3.STL; visual mesh filename=package://meshes/link3.STL
- added link left_link4, mass 0.127087; collision mesh filename=package://meshes/link4.STL; visual mesh filename=package://meshes/link4.STL
- added link left_link5, mass 0.144711; collision mesh filename=package://meshes/link5.STL; visual mesh filename=package://meshes/link5.STL
- added link left_link6, mass 0.195187; collision mesh filename=package://meshes/link6.STL; visual mesh filename=package://meshes/link6.STL
- added link left_link7, mass 0.0264823; collision mesh filename=package://meshes/link7.STL; visual mesh filename=package://meshes/link7.STL
- added link left_link8, mass 0.0264822; collision mesh filename=package://meshes/link8.STL; visual mesh filename=package://meshes/link8.STL
- added link right_base_link, mass 0.097868; collision mesh filename=package://meshes/base_link.STL; visual mesh filename=package://meshes/base_link.STL
- added link right_camera_link, mass 0.001; visual box size=0.01 0.01 0.01
- added link right_link1, mass 0.097868; collision mesh filename=package://meshes/link1.STL; visual mesh filename=package://meshes/link1.STL
- added link right_link2, mass 0.290889; collision mesh filename=package://meshes/link2.STL; visual mesh filename=package://meshes/link2.STL
- added link right_link3, mass 0.290848; collision mesh filename=package://meshes/link3.STL; visual mesh filename=package://meshes/link3.STL
- added link right_link4, mass 0.127087; collision mesh filename=package://meshes/link4.STL; visual mesh filename=package://meshes/link4.STL
- added link right_link5, mass 0.144711; collision mesh filename=package://meshes/link5.STL; visual mesh filename=package://meshes/link5.STL
- added link right_link6, mass 0.195187; collision mesh filename=package://meshes/link6.STL; visual mesh filename=package://meshes/link6.STL
- added link right_link7, mass 0.0264823; collision mesh filename=package://meshes/link7.STL; visual mesh filename=package://meshes/link7.STL
- added link right_link8, mass 0.0264822; collision mesh filename=package://meshes/link8.STL; visual mesh filename=package://meshes/link8.STL
- link base_link: geometry collision mesh filename=package://meshes/base_link_aloha.STL; visual mesh filename=package://meshes/base_link_aloha.STL
Joints:
- removed joint base_to_dummy
- removed joint joint1
- removed joint joint2
- removed joint joint3
- removed joint joint4
- removed joint joint5
- removed joint joint6
- removed joint joint6_to_gripper_base
- removed joint joint7
- removed joint joint8
- added joint base_to_left_base: type fixed, parent base_link, child left_base_link, origin xyz=0.234 0.303 0.761 rpy=0 0 0
- added joint base_to_right_base: type fixed, parent base_link, child right_base_link, origin xyz=0.234 -0.303 0.761 rpy=0 0 0
- added joint left_camera_joint: type fixed, parent left_link6, child left_camera_link, origin xyz=0.0 0.08 -0.0 rpy=0.5 3.14 0
- added joint left_elbow: type revolute, parent left_link2, child left_link3, origin xyz=0.28358 0.028726 0 rpy=0 0 -1.7939, axis 0 0 1, limit lower=-2.697 upper=0 effort=100 velocity=5
- added joint left_forearm_roll: type revolute, parent left_link3, child left_link4, origin xyz=-0.24221 0.068514 0 rpy=1.5708 0 0, axis 0 0 1, limit lower=-1.832 upper=1.832 effort=100 velocity=5
- added joint left_left_finger: type prismatic, parent left_link6, child left_link7, origin xyz=0 0 0.13503 rpy=1.5708 0 0, axis 0 0 -1, limit lower=0 upper=0.04 effort=100 velocity=1
- added joint left_right_finger: type prismatic, parent left_link6, child left_link8, origin xyz=0 0 0.13503 rpy=1.5708 0 -3.1416, axis 0 0 1, limit lower=-0.04 upper=0 effort=100 velocity=1
- added joint left_shoulder: type revolute, parent left_link1, child left_link2, origin xyz=0 0 0 rpy=1.5708 -0.1359 -3.1416, axis 0 0 1, limit lower=0 upper=3.14 effort=100 velocity=5
- added joint left_waist: type revolute, parent left_base_link, child left_link1, origin xyz=0 0 0.123 rpy=0 0 0, axis 0 0 1, limit lower=-2.618 upper=2.618 effort=100 velocity=5
- added joint left_wrist_angle: type revolute, parent left_link4, child left_link5, origin xyz=0 0 0 rpy=-1.5708 0 0, axis 0 0 1, limit lower=-1.22 upper=1.22 effort=100 velocity=5
- added joint left_wrist_rotate: type revolute, parent left_link5, child left_link6, origin xyz=0 0.091 0.0014165 rpy=1.5708 0 0, axis 0 0 1, limit lower=-3.14 upper=3.14 effort=100 velocity=5
- added joint right_camera_joint: type fixed, parent right_link6, child right_camera_link, origin xyz=0.0 0.08 -0.0 rpy=0.5 3.14 0
- added joint right_elbow: type revolute, parent right_link2, child right_link3, origin xyz=0.28358 0.028726 0 rpy=0 0 -1.7939, axis 0 0 1, limit lower=-2.697 upper=0 effort=100 velocity=5
- added joint right_forearm_roll: type revolute, parent right_link3, child right_link4, origin xyz=-0.24221 0.068514 0 rpy=1.5708 0 0, axis 0 0 1, limit lower=-1.832 upper=1.832 effort=100 velocity=5
- added joint right_left_finger: type prismatic, parent right_link6, child right_link7, origin xyz=0 0 0.13503 rpy=1.5708 0 0, axis 0 0 -1, limit lower=0 upper=0.04 effort=100 velocity=1
- added joint right_right_finger: type prismatic, parent right_link6, child right_link8, origin xyz=0 0 0.13503 rpy=1.5708 0 -3.1416, axis 0 0 1, limit lower=-0.04 upper=0 effort=100 velocity=1
- added joint right_shoulder: type revolute, parent right_link1, child right_link2, origin xyz=0 0 0 rpy=1.5708 -0.1359 -3.1416, axis 0 0 1, limit lower=0 upper=3.14 effort=100 velocity=5
- added joint right_waist: type revolute, parent right_base_link, child right_link1, origin xyz=0 0 0.123 rpy=0 0 0, axis 0 0 1, limit lower=-2.618 upper=2.618 effort=100 velocity=5
- added joint right_wrist_angle: type revolute, parent right_link4, child right_link5, origin xyz=0 0 0 rpy=-1.5708 0 0, axis 0 0 1, limit lower=-1.22 upper=1.22 effort=100 velocity=5
- added joint right_wrist_rotate: type revolute, parent right_link5, child right_link6, origin xyz=0 0.091 0.0014165 rpy=1.5708 0 0, axis 0 0 1, limit lower=-3.14 upper=3.14 effort=100 velocity=5
